Commit message: Add initial SRDFs
Use primitive cylinders for camera mast and drop mast meshes
Bump robotiq dep for new finger design

File: robots/common/cortado_cart.xacro (robot description, xacro)
@@ -36,14 +36,14 @@
             </inertial>
             <visual>
-                <origin xyz="-0.036 0.200134 0.00244588" rpy="0 0 0" />
-                <geometry>
-                    <mesh filename="package://cortado_description/meshes/camera_mast.gltf" scale="1 1 1" />
+                <origin xyz="0.175 0 0" rpy="0 1.5708 0" />
+                <geometry>
+                    <cylinder radius="0.014075" length="0.35" />
                 </geometry>
                 <material name="dark_gray_plastic" />
             </visual>
-            <collision name="box_collision_1">
-                <origin xyz="0.1775 0 0" rpy="0 0 0" />
-                <geometry>
-                    <box size="0.355 0.057 0.057" />
+            <collision name="cylinder_collision_1">
+                <origin xyz="0.175 0 0" rpy="0 1.5708 0" />
+                <geometry>
+                    <cylinder radius="0.014075" length="0.35" />
                 </geometry>
             </collision>
@@ -58,14 +58,14 @@
             </inertial>
             <visual>
-                <origin xyz="-0.391 0.200134 0.00244588" rpy="0 0 0" />
-                <geometry>
-                    <mesh filename="package://cortado_description/meshes/camera_mast_extension.gltf" scale="1 1 1" />
+                <origin xyz="0.175 0 0" rpy="0 1.5708 0" />
+                <geometry>
+                    <cylinder radius="0.014075" length="0.35" />
                 </geometry>
                 <material name="dark_gray_plastic" />
             </visual>
-            <collision name="box_collision_1">
-                <origin xyz="0.175 0 0" rpy="0 0 0" />
-                <geometry>
-                    <box size="0.35 0.015 0.015" />
+            <collision name="cylinder_collision_1">
+                <origin xyz="0.175 0 0" rpy="0 1.5708 0" />
+                <geometry>
+                    <cylinder radius="0.014075" length="0.35" />
                 </geometry>
             </collision>
@@ -3241,5 +3241,5 @@
         <xacro:if value="${int(camera_mast) >= 2}">
         <joint name="${pp}camera_mast_to_camera_mast_extension_joint" type="fixed">
-            <origin xyz="0.355 0 0" rpy="0 0 0" />
+            <origin xyz="0.35 0 0" rpy="0 0 0" />
             <axis xyz="-1 0 0" />
             <parent link="${pp}camera_mast" />

File: robots/common/fr3_robotiq_2f_85.xacro (robot description, xacro)
@@ -49,5 +49,5 @@
       </geometry>
       <material name="">
-        <color rgba="0.1 0.1 0.1 1" />
+        <color rgba="0.13 0.13 0.13 1" />
       </material>
     </visual>

File: robots/cortado.urdf.xacro (robot description, xacro)
@@ -7,5 +7,5 @@
   <xacro:arg name="wrist_camera" default="true" />
   <xacro:arg name="flip_gripper" default="true" />
-  <xacro:include filename="../urdf/cortado.urdf.xacro" />
+  <xacro:include filename="common/cortado.xacro" />
   <xacro:cortado
     prefix="$(arg prefix)"

File: robots/fr3_robotiq_2f_85.urdf.xacro (robot description, xacro)
@@ -6,5 +6,5 @@
   <xacro:arg name="wrist_camera" default="true" />
   <xacro:arg name="flip_gripper" default="true" />
-  <xacro:include filename="../urdf/fr3_robotiq_2f_85.urdf.xacro" />
+  <xacro:include filename="common/fr3_robotiq_2f_85.xacro" />
   <xacro:fr3_robotiq_2f_85
     prefix="$(arg prefix)"
